File: mk0.kicad_sch (KiCad schematic)
At the start: 26 parts, among them J1 USB_C_Receptacle_USB2.0_16P, J2 AudioJack4, J3 Conn_ARM_JTAG_SWD_10, SW1 SW_RESET, SW2 SW_BOOT, U1 LM3480-3.3, U2 STM32F072CBTx, Y1 8MHz

Commit message: Finish routing for switches
Connections:
- net Col4: now also U2.42 (PB6); no longer U2.45 (PB8)
- net Col5: now also U2.43 (PB7); no longer U2.46 (PB9)
- net Col6: now also U2.45 (PB8); no longer U2.21 (PB10)
- net Row0: now also U2.17 (PA7); no longer U2.18 (PB0)
- net Row1: now also U2.18 (PB0); no longer U2.19 (PB1)
- net Row2: now also U2.19 (PB1); no longer U2.20 (PB2)
- net Row3: now also U2.20 (PB2); no longer U2.22 (PB11)
- net Row4: now also U2.22 (PB11); no longer U2.25 (PB12)
