File: right/matrix.kicad_sch (KiCad schematic)
At the start: 66 parts, among them SW10 tab, SW11 q, SW12 w, SW13 e, SW14 r, SW15 t, SW16 [, SW17 caps, SW18 a, SW19 s, SW20 d, SW21 f, SW22 g, SW23 ->, SW24 shift, SW25 z, SW26 x, SW27 c, SW28 v, SW29 b, SW3 `, SW30 custom2, SW31 ctrl, SW32 menu, SW33 alt, SW34 space, SW35 space, SW4 1, SW5 2, SW6 3, SW7 4, SW8 5, SW9 -

Commit message: Finish right halve
Parts:
- SW24: value shift -> z
Changed lines of the file:
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@@
 	)
 	(junction
+		(at 45.72 105.41)
+		(diameter 0)
+		(color 0 0 0 0)
+	)
+	(junction
 		(at 198.12 105.41)
 		(diameter 0)
@@
 	)
 	(junction
-		(at 45.72 105.41)
-		(diameter 0)
-		(color 0 0 0 0)
-	)
-	(junction
 		(at 161.29 85.09)
 		(diameter 0)
@@
 	(wire
 		(pts
-			(xy 45.72 105.41) (xy 45.72 115.57)
-		)
-		(stroke
-			(width 0)
-			(type default)
-		)
-	)
-	(wire
-		(pts
 			(xy 45.72 85.09) (xy 45.72 95.25)
 		)
@@
 	(wire
 		(pts
+			(xy 45.72 105.41) (xy 45.72 115.57)
+		)
+		(stroke
+			(width 0)
+			(type default)
+		)
+	)
+	(wire
+		(pts
 			(xy 276.86 74.93) (xy 276.86 85.09)
 		)
@@
 		)
 	)
-	(global_label "Row3"
+	(global_label "Row4"
 		(shape input)
-		(at 27.94 105.41 180)
+		(at 106.68 115.57 180)
 		(fields_autoplaced yes)
 		(effects
@@
 		)
 		(property "Intersheetrefs" "${INTERSHEET_REFS}"
-			(at 19.9958 105.41 0)
+			(at 98.7358 115.57 0)
 			(effects
 				(font
@@
 		)
 	)
-	(global_label "Row4"
+	(global_label "Col0"
 		(shape input)
-		(at 106.68 115.57 180)
+		(at 45.72 74.93 0)
 		(fields_autoplaced yes)
 		(effects
@@
 				(size 1.27 1.27)
 			)
-			(justify right)
+			(justify left)
 		)
 		(property "Intersheetrefs" "${INTERSHEET_REFS}"
-			(at 98.7358 115.57 0)
+			(at 52.9989 74.93 0)
 			(effects
 				(font
 					(size 1.27 1.27)
 				)
-				(justify right)
+				(justify left)
 				(hide yes)
 			)
 		)
 	)
-	(global_label "Col0"
+	(global_label "Row3"
 		(shape input)
-		(at 45.72 74.93 0)
+		(at 27.94 105.41 180)
 		(fields_autoplaced yes)
 		(effects
@@
 				(size 1.27 1.27)
 			)
-			(justify left)
+			(justify right)
 		)
 		(property "Intersheetrefs" "${INTERSHEET_REFS}"
-			(at 52.9989 74.93 0)
+			(at 19.9958 105.41 0)
 			(effects
 				(font
 					(size 1.27 1.27)
 				)
-				(justify left)
+				(justify right)
 				(hide yes)
 			)
@@
 	)
 	(symbol
+		(lib_id "Device:D")
+		(at 31.75 105.41 0)
+		(unit 1)
+		(exclude_from_sim no)
+		(in_bom yes)
+		(on_board yes)
+		(dnp no)
+		(fields_autoplaced yes)
+		(property "Reference" "D22"
+			(at 31.75 99.06 0)
+			(effects
+				(font
+					(size 1.27 1.27)
+				)
+			)
+		)
+		(property "Value" "D"
+			(at 31.75 101.6 0)
+			(effects
+				(font
+					(size 1.27 1.27)
+				)
+			)
+		)
+		(property "Footprint" "Diode_SMD:D_SOD-323_HandSoldering"
+			(at 31.75 105.41 0)
+			(effects
+				(font
+					(size 1.27 1.27)
+				)
+				(hide yes)
+			)
+		)
+		(property "Datasheet" "~"
+			(at 31.75 105.41 0)
+			(effects
+				(font
+					(size 1.27 1.27)
+				)
+				(hide yes)
+			)
+		)
+		(property "Description" "Diode"
+			(at 31.75 105.41 0)
+			(effects
+				(font
+					(size 1.27 1.27)
+				)
+				(hide yes)
+			)
+		)
+		(property "Sim.Device" "D"
+			(at 31.75 105.41 0)
+			(effects
+				(font
+					(size 1.27 1.27)
+				)
+				(hide yes)
+			)
+		)
+		(property "Sim.Pins" "1=K 2=A"
+			(at 31.75 105.41 0)
+			(effects
+				(font
+					(size 1.27 1.27)
+				)
+				(hide yes)
+			)
+		)
+		(pin "2"
+		)
+		(pin "1"
+		)
+		(instances
+			(project "right"
+				(path "/bdb963a7-1785-4642-8248-f83dad46c2d3/6aba7e77-b5f5-4af6-8cbc-f75bd0f2a691"
+					(reference "D22")
+					(unit 1)
+				)
+			)
+		)
+	)
+	(symbol
 		(lib_id "Switch:SW_Push")
 		(at 40.64 95.25 0)
@@
 	(symbol
 		(lib_id "Device:D")
-		(at 31.75 105.41 0)
-		(unit 1)
-		(exclude_from_sim no)
-		(in_bom yes)
-		(on_board yes)
-		(dnp no)
-		(fields_autoplaced yes)
-		(property "Reference" "D22"
-			(at 31.75 99.06 0)
-			(effects
-				(font
-					(size 1.27 1.27)
-				)
-			)
-		)
-		(property "Value" "D"
-			(at 31.75 101.6 0)
-			(effects
-				(font
-					(size 1.27 1.27)
-				)
-			)
-		)
-		(property "Footprint" "Diode_SMD:D_SOD-323_HandSoldering"
-			(at 31.75 105.41 0)
-			(effects
-				(font
-					(size 1.27 1.27)
-				)
-				(hide yes)
-			)
-		)
-		(property "Datasheet" "~"
-			(at 31.75 105.41 0)
-			(effects
-				(font
-					(size 1.27 1.27)
-				)
-				(hide yes)
-			)
-		)
-		(property "Description" "Diode"
-			(at 31.75 105.41 0)
-			(effects
-				(font
-					(size 1.27 1.27)
-				)
-				(hide yes)
-			)
-		)
-		(property "Sim.Device" "D"
-			(at 31.75 105.41 0)
-			(effects
-				(font
-					(size 1.27 1.27)
-				)
-				(hide yes)
-			)
-		)
-		(property "Sim.Pins" "1=K 2=A"
-			(at 31.75 105.41 0)
-			(effects
-				(font
-					(size 1.27 1.27)
-				)
-				(hide yes)
-			)
-		)
-		(pin "2"
-		)
-		(pin "1"
-		)
-		(instances
-			(project "right"
-				(path "/bdb963a7-1785-4642-8248-f83dad46c2d3/6aba7e77-b5f5-4af6-8cbc-f75bd0f2a691"
-					(reference "D22")
-					(unit 1)
-				)
-			)
-		)
-	)
-	(symbol
-		(lib_id "Device:D")
 		(at 220.98 95.25 0)
 		(unit 1)
@@
 	(symbol
 		(lib_id "Switch:SW_Push")
-		(at 40.64 105.41 0)
+		(at 119.38 95.25 0)
 		(unit 1)
 		(exclude_from_sim no)
@@
 		(dnp no)
 		(fields_autoplaced yes)
-		(property "Reference" "SW24"
-			(at 40.64 97.79 0)
+		(property "Reference" "SW19"
+			(at 119.38 87.63 0)
 			(effects
 				(font
@@
 			)
 		)
-		(property "Value" "shift"
-			(at 40.64 100.33 0)
+		(property "Value" "s"
+			(at 119.38 90.17 0)
 			(effects
 				(font
@@
 			)
 		)
-		(property "Footprint" "Button_Switch_Keyboard:SW_Cherry_MX_2.00u_Plate"
-			(at 40.64 100.33 0)
+		(property "Footprint" "Button_Switch_Keyboard:SW_Cherry_MX_1.00u_Plate"
+			(at 119.38 90.17 0)
 			(effects
 				(font
@@
 		)
 		(property "Datasheet" "~"
-			(at 40.64 100.33 0)
+			(at 119.38 90.17 0)
 			(effects
 				(font
@@
 		)
 		(property "Description" "Push button switch, generic, two pins"
-			(at 40.64 105.41 0)
+			(at 119.38 95.25 0)
 			(effects
 				(font
@@
 			(project "right"
 				(path "/bdb963a7-1785-4642-8248-f83dad46c2d3/6aba7e77-b5f5-4af6-8cbc-f75bd0f2a691"
-					(reference "SW24")
+					(reference "SW19")
 					(unit 1)
 				)
@@
 	(symbol
 		(lib_id "Switch:SW_Push")
-		(at 119.38 95.25 0)
+		(at 40.64 105.41 0)
 		(unit 1)
 		(exclude_from_sim no)
@@
 		(dnp no)
 		(fields_autoplaced yes)
-		(property "Reference" "SW19"
-			(at 119.38 87.63 0)
+		(property "Reference" "SW24"
+			(at 40.64 97.79 0)
 			(effects
 				(font
@@
 			)
 		)
-		(property "Value" "s"
-			(at 119.38 90.17 0)
+		(property "Value" "z"
+			(at 40.64 100.33 0)
 			(effects
 				(font
@@
 			)
 		)
-		(property "Footprint" "Button_Switch_Keyboard:SW_Cherry_MX_1.00u_Plate"
-			(at 119.38 90.17 0)
+		(property "Footprint" "Button_Switch_Keyboard:SW_Cherry_MX_2.00u_Plate"
+			(at 40.64 100.33 0)
 			(effects
 				(font
@@
 		)
 		(property "Datasheet" "~"
-			(at 119.38 90.17 0)
+			(at 40.64 100.33 0)
 			(effects
 				(font
@@
 		)
 		(property "Description" "Push button switch, generic, two pins"
-			(at 119.38 95.25 0)
+			(at 40.64 105.41 0)
 			(effects
 				(font
@@
 			(project "right"
 				(path "/bdb963a7-1785-4642-8248-f83dad46c2d3/6aba7e77-b5f5-4af6-8cbc-f75bd0f2a691"
-					(reference "SW19")
+					(reference "SW24")
 					(unit 1)
 				)
