File: right/right.kicad_sch (KiCad schematic)
At the start: 26 parts, among them J1 USB_C_Receptacle_USB2.0_16P, J2 AudioJack4, J3 Conn_ARM_JTAG_SWD_10, SW1 SW_RESET, SW2 SW_BOOT, U1 LM3480-3.3, U2 STM32F072CBTx, Y1 8MHz

Commit message: change cristals
Parts:
- removed R4: 390, Resistor_SMD:R_0805_2012Metric_Pad1.20x1.40mm_HandSolder, symbol Device:R
- removed Y1: 8MHz, Crystal:Crystal_SMD_2012-2Pin_2.0x1.2mm_HandSoldering, symbol Device:Crystal
- added Y1: 8MHz, Crystal:Crystal_SMD_3225-4Pin_3.2x2.5mm_HandSoldering, symbol Device:Crystal_GND24_Small
Connections:
- net GND: now also Y1.2, Y1.4
- net at C13.1, U2.5 (PF0): now also Y1.1
- net at U2.6 (PF1): now also C14.1, Y1.3
